Commit message: Add SO101 teleoperation and PAROL6 demonstration collection
Map a calibrated SO101 leader pose to PAROL6 Cartesian targets with configurable frame transforms and gripper control. Add package launch files and native LeRobot episode recording with start, save and discard services.

Add a cube, container and contact jaws to the simulation, align the robot mounting frame, and scope Foxglove launch arguments so its port cannot override the leader serial port.

File: src/robot_server/assets/parol6/parol6.urdf (robot description, URDF)
Before this commit: robot parol6, 12 links, 11 joints
Joints:
- joint base_joint: origin xyz=0.0 0.0 0.00 rpy=0 0 0 -> xyz=0.0 0.0 0.00 rpy=0 0 -1.5707963267948966

Commit message: Fixes

File: src/robot_server/assets/parol6/parol6.urdf (robot description, URDF)
Before this commit: robot parol6, 12 links, 11 joints
Joints:
- joint base_joint: origin xyz=0.0 0.0 0.00 rpy=0 0 -1.5707963267948966 -> xyz=0.0 0.0 0.00 rpy=0 0 0
