Commit message: telop mujoco for so101 and parol6 working

File: src/robot_description/robot_description/assets/deferred/parol6/parol6.urdf (robot description, URDF)
Before this commit: robot parol6, 12 links, 11 joints
Links:
- link base_link: geometry collision mesh filename=package://robot_description/deferred/parol6/meshes/base_lin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; visual mesh filename=package://robot_description/deferred/parol6/meshes/base_lin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
- link link_1: geometry collision mesh filename=package://robot_description/deferred/parol6/meshes/L1_simpl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; visual mesh filename=package://robot_description/deferred/parol6/meshes/L1.STL
- link link_2: geometry collision mesh filename=package://robot_description/deferred/parol6/meshes/L2_simpl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; visual mesh filename=package://robot_description/deferred/parol6/meshes/L2.STL
- link link_3: geometry collision mesh filename=package://robot_description/deferred/parol6/meshes/L3_simpl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; visual mesh filename=package://robot_description/deferred/parol6/meshes/L3.STL
- link link_4: geometry collision mesh filename=package://robot_description/deferred/parol6/meshes/L4_simpl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; visual mesh filename=package://robot_description/deferred/parol6/meshes/L4.STL
- link link_5: geometry collision mesh filename=package://robot_description/deferred/parol6/meshes/L5_simpl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; visual mesh filename=package://robot_description/deferred/parol6/meshes/L5.STL
- link link_6: geometry collision mesh filename=package://robot_description/deferred/parol6/meshes/L6_simpl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; visual mesh filename=package://robot_description/deferred/parol6/meshes/L6.STL
- link tool_body: geometry collision mesh filename=package://robot_description/deferred/parol6/meshes/pneumati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; visual mesh filename=package://robot_description/deferred/parol6/meshes/pneumati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
- link tool_left_jaw: geometry collision mesh filename=package://robot_description/deferred/parol6/meshes/pneumati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; visual mesh filename=package://robot_description/deferred/parol6/meshes/pneumati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
- link tool_right_jaw: geometry collision mesh filename=package://robot_description/deferred/parol6/meshes/pneumati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; visual mesh filename=package://robot_description/deferred/parol6/meshes/pneumati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
Joints:
- removed joint tool_right_jaw_joint
- added joint gripper_slide: type prismatic, parent link_6, child tool_right_jaw, origin xyz=0 0 0 rpy=0 0 0, axis 0 1 0, limit lower=0 upper=0.0035 effort=10 velocity=0.1
